File: hardware/overview/motor_interface.kicad_sch (KiCad schematic)
At the start: 3 parts

Commit message: schematics
Parts:
- removed U1: (no value), symbol kl_parts:kl_amistar_hio_CN2
- removed U3: (no value), symbol kl_parts:CNC4PC
- added 75ALS1, 75ALS2: (no value), symbol kl_parts:75ALS171
- added D1: 1N5401, Diode_THT:D_DO-201AD_P15.24mm_Horizontal, symbol Diode:1N5401
- added DYN1, DYN2: (no value), symbol kl_parts:DYN4
Connections:
- net at U2. (COM): now also D1.1 (K)
- net at U2.2 (parport_2): now also 75ALS1.8 (2D)
- net at U2.3 (parport_3): now also 75ALS1.3 (1D)
- net at U2.4 (parport_4): now also 75ALS2.3 (1D)
- net at U2.5 (parport_5): now also 75ALS1.11 (3D)
- new net: 75ALS1.13 (3B), DYN2.10 (DIR-)
- new net: 75ALS2.19 (1A), DYN2.11 (PUL+)
- new net: 75ALS1.12 (3A), DYN2.22 (DIR+)
- new net: 75ALS2.20 (1B), DYN2.23 (PUL-)
- new net: 75ALS1.14 (2A), DYN1.11 (PUL+)
- new net: 75ALS1.15 (2B), DYN1.23 (PUL-)
- new net: 75ALS1.19 (1A), DYN1.22 (DIR+)
- new net: 75ALS1.20 (1B), DYN1.10 (DIR-)
- new net +5V: 75ALS1.16 (Vcc), 75ALS1.17 (CDE), 75ALS2.16 (Vcc), 75ALS2.17 (CDE)
- new net GND: 75ALS1.4 (GND), 75ALS1.5 (GND), 75ALS2.4 (GND), 75ALS2.5 (GND), D1.2 (A), DYN1.1 (COM), DYN2.1 (COM)
Other:
- note added: "X AXIS"
- note added: "Y AXIS"
- note added: "attempt at noise cleanup"
- note added: "chip on left"
- note added: "chip on right"
