File: hardware/overview/logic_interface.kicad_sch (KiCad schematic)
At the start: 3 parts

Commit message: schematics
Parts:
- removed U1: (no value), symbol kl_parts:kl_amistar_hio_CN2
- added HIO_CN1: (no value), symbol kl_parts:kl_amistar_hio_CN1
- added HIO_CN2: (no value), symbol kl_parts:kl_amistar_hio_CN2
- added HIO_CN3: (no value), symbol kl_parts:kl_amistar_hio_CN3
- added HIO_RU1: (no value), symbol kl_parts:kl_amistar_hio_RU

Commit message: schematics
Parts:
- removed U3: (no value), symbol kl_parts:CNC4PC
Other:
- note added: "HIO power"
- moved on the sheet: HIO_CN1
Changed lines of the file:
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@@
 	(generator_version "10.0")
 	(paper "A4")
+	(text "HIO power"
+		(exclude_from_sim no)
+		(at 223.012 26.67 0)
+		(effects
+			(font
+				(size 1.27 1.27)
+			)
+		)
+	)
 	(symbol
 		(lib_id "kl_parts:kl_amistar_hio_CN3")
@@
 	(symbol
 		(lib_id "kl_parts:kl_amistar_hio_CN1")
-		(at 209.55 40.64 0)
+		(at 223.52 40.64 0)
 		(unit 1)
 		(body_style 1)
@@
 		(fields_autoplaced yes)
 		(property "Reference" "HIO_CN1"
-			(at 219.71 44.4499 0)
+			(at 233.68 44.4499 0)
 			(show_name no)
 			(do_not_autoplace no)
@@
 		)
 		(property "Value" ""
-			(at 209.55 40.64 0)
+			(at 223.52 40.64 0)
 			(show_name no)
 			(do_not_autoplace no)
@@
 		)
 		(property "Footprint" ""
-			(at 209.55 40.64 0)
+			(at 223.52 40.64 0)
 			(hide yes)
 			(show_name no)
@@
 		)
 		(property "Datasheet" ""
-			(at 209.55 40.64 0)
+			(at 223.52 40.64 0)
 			(hide yes)
 			(show_name no)
@@
 		)
 		(property "Description" ""
-			(at 209.55 40.64 0)
+			(at 223.52 40.64 0)
 			(hide yes)
 			(show_name no)
@@
 					(unit 1)
 				)
-			)
-		)
-	)
-	(symbol
-		(lib_name "CNC4PC_1")
-		(lib_id "kl_parts:CNC4PC")
-		(at 30.48 168.91 0)
-		(unit 1)
-		(body_style 1)
-		(exclude_from_sim no)
-		(in_bom yes)
-		(on_board yes)
-		(in_pos_files yes)
-		(dnp no)
-		(fields_autoplaced yes)
-		(property "Reference" "U3"
-			(at 30.48 168.91 0)
-			(hide yes)
-			(show_name no)
-			(do_not_autoplace no)
-			(effects
-				(font
-					(size 1.27 1.27)
-				)
-			)
-		)
-		(property "Value" ""
-			(at 30.48 168.91 0)
-			(show_name no)
-			(do_not_autoplace no)
-			(effects
-				(font
-					(size 1.27 1.27)
-				)
-			)
-		)
-		(property "Footprint" ""
-			(at 30.48 168.91 0)
-			(hide yes)
-			(show_name no)
-			(do_not_autoplace no)
-			(effects
-				(font
-					(size 1.27 1.27)
-				)
-			)
-		)
-		(property "Datasheet" ""
-			(at 30.48 168.91 0)
-			(hide yes)
-			(show_name no)
-			(do_not_autoplace no)
-			(effects
-				(font
-					(size 1.27 1.27)
-				)
-			)
-		)
-		(property "Description" ""
-			(at 30.48 168.91 0)
-			(hide yes)
-			(show_name no)
-			(do_not_autoplace no)
-			(effects
-				(font
-					(size 1.27 1.27)
-				)
-			)
-		)
-		(pin "9"
-		)
-		(pin "13"
-		)
-		(pin "6"
-		)
-		(pin ""
-		)
-		(pin ""
-		)
-		(pin ""
-		)
-		(pin "11"
-		)
-		(pin "17"
-		)
-		(pin "15"
-		)
-		(pin "10"
-		)
-		(pin "16"
-		)
-		(pin "2"
-		)
-		(pin "3"
-		)
-		(pin "8"
-		)
-		(pin "1"
-		)
-		(pin "5"
-		)
-		(pin "12"
-		)
-		(pin "4"
-		)
-		(pin "7"
-		)
-		(pin "14"
-		)
-		(instances
-			(project "logic_interface"
-				(path "/d999ca8c-b4a1-4c29-819a-63809fda4f99"
-					(reference "U3")
-					(unit 1)
-				)

Commit message: schematics
Parts:
- added D1: 1N5401, Diode_THT:D_DO-201AD_P15.24mm_Horizontal, symbol Diode:1N5401
Connections:
- net GND: now reaches U2. (COM)
- net GND: now also D1.2 (A)
- new net: D1.1 (K), U2. (COM)
- new net +5V: U2. (COM)
Other:
- note added: "ORIG HIO"
- note added: "attempt at noise cleanup"
- moved on the sheet: HIO_CN1, HIO_CN2, HIO_CN3, HIO_RU1
