File: hardware/overview/hio_second_brd.kicad_sch (KiCad schematic)
At the start: 3 parts

Commit message: schematics
Parts:
- renumbered HIO_CN4 to HIO_CN1, HIO_CN5 to HIO_CN2, HIO_CN6 to HIO_CN3
Changed lines of the file:
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@@
 		(dnp no)
 		(fields_autoplaced yes)
-		(property "Reference" "HIO_CN4"
+		(property "Reference" "HIO_CN1"
 			(at 31.9968 20.32 0)
 			(show_name no)
@@
 		)
 		(instances
-			(project "hio_first_brd"
+			(project "hio_second_brd"
 				(path "/d999ca8c-b4a1-4c29-819a-63809fda4f99"
-					(reference "HIO_CN4")
+					(reference "HIO_CN1")
 					(unit 1)
 				)
@@
 		)
 		(instances
-			(project "hio_first_brd"
+			(project "hio_second_brd"
 				(path "/d999ca8c-b4a1-4c29-819a-63809fda4f99"
 					(reference "#PWR01")
@@
 		(dnp no)
 		(fields_autoplaced yes)
-		(property "Reference" "HIO_CN6"
+		(property "Reference" "HIO_CN3"
 			(at 35.1718 110.49 0)
 			(show_name no)
@@
 		)
 		(instances
-			(project "hio_first_brd"
+			(project "hio_second_brd"
 				(path "/d999ca8c-b4a1-4c29-819a-63809fda4f99"
-					(reference "HIO_CN6")
+					(reference "HIO_CN3")
 					(unit 1)
 				)
@@
 		)
 		(instances
-			(project "hio_first_brd"
+			(project "hio_second_brd"
 				(path "/d999ca8c-b4a1-4c29-819a-63809fda4f99"
 					(reference "#PWR02")
@@
 		)
 		(instances
-			(project "hio_first_brd"
+			(project "hio_second_brd"
 				(path "/d999ca8c-b4a1-4c29-819a-63809fda4f99"
 					(reference "#PWR03")
@@
 		(dnp no)
 		(fields_autoplaced yes)
-		(property "Reference" "HIO_CN5"
+		(property "Reference" "HIO_CN2"
 			(at 46.355 58.42 0)
 			(show_name no)
@@
 		)
 		(instances
-			(project "hio_first_brd"
+			(project "hio_second_brd"
 				(path "/d999ca8c-b4a1-4c29-819a-63809fda4f99"
-					(reference "HIO_CN5")
+					(reference "HIO_CN2")
 					(unit 1)
 				)

Commit message: schematics
Parts:
- added 75ALS1: (no value), symbol kl_parts:75ALS171
- added C1, C2: C, symbol Device:C
- added C3: C_Polarized, symbol Device:C_Polarized
- added D1, D2, D3, D4, D5: LED, symbol Device:LED
- added D6: st7735_tft, symbol kl_parts:st7735_tft
- added R1: R, symbol Device:R
- added U1: ATmega2560-16A, Package_QFP:TQFP-100_14x14mm_P0.5mm, symbol MCU_Microchip_ATmega:ATmega2560-16A
Connections:
- net +5V: now also HIO_CN3.2 (power), 75ALS1.16 (Vcc), C1.1, C2.1, C3.1, D5.2 (A), U1.10 (VCC), U1.100 (AVCC), U1.31 (VCC), U1.61 (VCC), U1.80 (VCC)
- net GND: now also HIO_CN3.1 (GND), 75ALS1.4 (GND), 75ALS1.5 (GND), C1.2, C2.2, C3.2, D1.1 (K), D2.1 (K), D3.1 (K), D4.1 (K), R1.2
- new net: D4.2 (A), HIO_CN3.6 (vacuum-s)
- new net: D3.2 (A), HIO_CN3.5 (vacuum-s)
- new net: D5.1 (K), R1.1
- new net: U1.11 (GND), U1.32 (GND), U1.62 (GND), U1.81 (GND), U1.99 (GND)
- new net: 75ALS1.19 (1A), HIO_CN2.1 (RD-)
- new net: 75ALS1.20 (1B), HIO_CN2.2 (RD+)
- new net: D2.2 (A), HIO_CN3.4 (vacuum-s)
- new net: D1.2 (A), HIO_CN3.3 (vacuum-s)
Other:
- note added: "HIO 12V is only 5V here!"
- note added: "pwr led"
